Commit message: Add robot arm joint dimension configuration

File: pwa-dobot-plc/robotarmv3-pi-service/demo-kinematics.urdf (robot description, URDF)
Before this commit: robot five_dof_arm, 7 links, 6 joints
Links:
- added link link6
Joints:
- added joint joint6_wrist_yaw: type revolute, parent link5, child link6, origin xyz=0.03 0 0 rpy=0 0 0, axis 0 0 1, limit lower=-3.14 upper=3.14 effort=5 velocity=3
- joint tool_fixed: parent link5 -> link6

Commit message: robot arm j6 added

File: pwa-dobot-plc/robotarmv3-pi-service/demo-kinematics.urdf (robot description, URDF)
Before this commit: robot six_dof_arm, 8 links, 7 joints
Joints:
- joint joint6_wrist_yaw: origin xyz=0.03 0 0 rpy=0 0 0 -> xyz=0.042 0 0 rpy=0 0 0
- joint tool_fixed: origin xyz=0.042 0 0 rpy=0 0 0 -> xyz=0.083 0 0 rpy=0 0 0
