Commit message: Update arm bridge to upstream RobotArmv3 013a1a9 (+ PORT/BAUD env edits)
app/robotarmv3-pi-service is now Ben's raspberry-pi-control-st3215 as of
2026-10-21 plus the two local edits recorded in LOCAL_PATCHES.md: PORT from env
(default 8090) and SERIAL_BAUDRATE from env. Removed stale installer files and
API_DOCUMENTATION.md; serialport 13 (package.json / lock). The mirror folder
raspberry-pi-control-st3215 is now pristine (UPSTREAM.md).

NOTE: the URDF changed (J1/J4 mirrored, link offsets, TCP lengths): stored XYZ
positions (home waypoint, DB125 pickup/pallet/quarantine) must be re-taught.
See docs/BEN_UPDATE_INTEGRATION_PLAN.md section 7.

Co-Authored-By: Claude Sonnet 5.5 <noreply@anthropic.com>

File: app/robotarmv3-pi-service/kinematics.urdf (robot description, URDF)
Before this commit: robot matrix_arm_v3, 12 links, 11 joints
Joints:
- joint joint1_base_yaw: axis 0 0 1 -> 0 0 -1; origin xyz=0 0 0.03538 rpy=0 0 0 -> xyz=0 0 0.036 rpy=0 0 0
- joint joint2_shoulder_pitch: origin xyz=0 0 0.08553 rpy=0 0 0 -> xyz=0 0 0.086 rpy=0 0 0
- joint joint3_elbow_pitch: origin xyz=0 0 0.11342 rpy=0 0 0 -> xyz=0 0 0.113 rpy=0 0 0
- joint joint4_wrist_roll: axis 1 0 0 -> -1 0 0
- joint joint6_wrist_roll_2: axis 1 0 0 -> 0 0 1
- joint tool_mount: origin xyz=0 0 -0.04463 rpy=0 0 0 -> xyz=0 0 -0.05 rpy=0 0 0
- joint tool_servo: origin xyz=0 0 -0.12019 rpy=0 0 0 -> xyz=0 0 -0.130 rpy=0 0 0
- joint tool_vacuum: origin xyz=0.00202 0 -0.11462 rpy=0 0 0 -> xyz=0.00202 0 -0.119 rpy=0 0 0
